File: PassiveAttenuator/PassiveAttenuator.kicad_pcb (KiCad board)
At the start: 2 copper layers, 15 x 100 mm, 6 parts, among them J1 AudioJack2_SwitchT, J2 AudioJack2_SwitchT, J3 AudioJack2_SwitchT, J4 AudioJack2_SwitchT

Commit message: Main PCB: add logo + harmonized branding text
This board had no logo at all. Added the medium S-mark plus
"schenktronics.com" and "ST-02 v1.0\nPassive Attenuator" in the clear
gap between the second jack and second pot -- the only real opening
given the pot footprints eat into the middle of the board.

Tried the CC BY-NC-SA roundels + text too, matching the Multiple, but
verified via kicad-cli renders that there isn't enough clear vertical
room between the pot's mounting pads and the jack above without
overlapping real copper -- left them off.
Parts:
- added G***: LOGO, _NTSFootprints:SchentronicsLogoSmed, B.Cu at (157.6, 98.0)
Other:
- board text added: "ST-02 v1.0 Passive Attenuator"
- board text removed: "Passive Attenuator v1.0"
Changed lines of the file:
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@@
     )
   )
-  (gr_text "Passive\nAttenuator\nv1.0" (at 164.25 100) (layer B.SilkS)
-    (effects (font (size 1 1) (thickness 0.15)) (justify left mirror))
-  )
-  (gr_text schenktronics.com (at 157.5 103.75) (layer B.SilkS)
-    (effects (font (size 1 1) (thickness 0.15)) (justify mirror))
-  )
+(footprint "_NTSFootprints:SchentronicsLogoSmed"
+		(layer "B.Cu")
+		(at 157.6 98.0 180)
+		(property "Reference" "G***"
+			(at 0 0 0)
+			(layer "B.SilkS")
+			(hide yes)
+			(effects
+				(font
+					(size 1.524 1.524)
+					(thickness 0.3)
+				)
+				(justify mirror)
+			)
+		)
+		(property "Value" "LOGO"
+			(at 0.75 0 0)
+			(layer "B.SilkS")
+			(hide yes)
+			(effects
+				(font
+					(size 1.524 1.524)
+					(thickness 0.3)
+				)
+				(justify mirror)
+			)
+		)
+		(property "Datasheet" ""
+			(at 0 0 0)
+			(layer "B.Fab")
+			(hide yes)
+			(effects
+				(font
+					(size 1.27 1.27)
+				)
+				(justify mirror)
+			)
+		)
+		(property "Description" ""
+			(at 0 0 0)
+			(layer "B.Fab")
+			(hide yes)
+			(effects
+				(font
+					(size 1.27 1.27)
+				)
+				(justify mirror)
+			)
+		)
+		(attr through_hole)
+		(duplicate_pad_numbers_are_jumpers no)
+		(fp_poly
+			(pts
+				(xy 1.868278 2.58143) (xy 1.996868 2.521286) (xy 2.139782 2.392248) (xy 2.141744 2.39023) (xy 2.26917 2.240218)
+				(xy 2.3282 2.104254) (xy 2.342016 1.940556) (xy 2.32674 1.76983) (xy 2.265128 1.636712) (xy 2.142578 1.49766)
+				(xy 1.99563 1.369822) (xy 1.860976 1.311314) (xy 1.705134 1.298434) (xy 1.477652 1.331602) (xy 1.282318 1.411322)
+				(xy 1.2077 1.451194) (xy 1.121914 1.480446) (xy 1.007106 1.500694) (xy 0.845422 1.513554) (xy 0.619012 1.52064)
+				(xy 0.310018 1.523564) (xy 0.036268 1.524) (xy -0.334734 1.52352) (xy -0.609672 1.520838) (xy -0.805376 1.5141)
+				(xy -0.93867 1.50145) (xy -1.026382 1.48103) (xy -1.085334 1.450982) (xy -1.132356 1.409454) (xy -1.1477 1.393362)
+				(xy -1.248618 1.216666) (xy -1.27943 1.004386) (xy -1.24152 0.797554) (xy -1.13628 0.637202) (xy -1.121706 0.624986)
+				(xy -1.063986 0.584848) (xy -0.996246 0.555086) (xy -0.901792 0.534162) (xy -0.763926 0.520532)
+				(xy -0.56595 0.512658) (xy -0.291166 0.508998) (xy 0.077122 0.508014) (xy 0.146178 0.508) (xy 0.541412 0.506826)
+				(xy 0.843058 0.502264) (xy 1.070404 0.492748) (xy 1.242738 0.47672) (xy 1.379344 0.452618) (xy 1.499512 0.418876)
+				(xy 1.574494 0.39233) (xy 1.909074 0.21196) (xy 2.1625 -0.043156) (xy 2.32748 -0.3624) (xy 2.396726 -0.735146)
+				(xy 2.39846 -0.808208) (xy 2.355202 -1.210738) (xy 2.223398 -1.54486) (xy 2 -1.81588) (xy 1.703516 -2.017972)
+				(xy 1.603364 -2.068812) (xy 1.51109 -2.107282) (xy 1.409074 -2.135422) (xy 1.279686 -2.15527) (xy 1.105304 -2.168868)
+				(xy 0.8683 -2.178252) (xy 0.551052 -2.185464) (xy 0.204482 -2.19142) (xy -0.202796 -2.199066) (xy -0.51338 -2.20787)
+				(xy -0.743462 -2.219324) (xy -0.909232 -2.234926) (xy -1.026886 -2.256166) (xy -1.112616 -2.284538)
+				(xy -1.178406 -2.318948) (xy -1.441264 -2.419342) (xy -1.709824 -2.414754) (xy -1.959414 -2.307126)
+				(xy -2.030464 -2.25193) (xy -2.152924 -2.130924) (xy -2.211672 -2.01751) (xy -2.229322 -1.859778)
+				(xy -2.229908 -1.801432) (xy -1.87427 -1.801432) (xy -1.86694 -1.85055) (xy -1.77418 -1.98203) (xy -1.623952 -2.041146)
+				(xy -1.45098 -2.02068) (xy -1.340984 -1.959882) (xy -1.273952 -1.8509) (xy -1.29005 -1.722216) (xy -1.372034 -1.605786)
+				(xy -1.502658 -1.533574) (xy -1.576156 -1.524) (xy -1.720106 -1.566822) (xy -1.83016 -1.671296)
+				(xy -1.87427 -1.801432) (xy -2.229908 -1.801432) (xy -2.229984 -1.793876) (xy -2.220208 -1.61113)
+				(xy -2.174986 -1.48651) (xy -2.070484 -1.365858) (xy -2.021398 -1.319946) (xy -1.793456 -1.172918)
+				(xy -1.55048 -1.122256) (xy -1.316934 -1.170282) (xy -1.198582 -1.241778) (xy -1.143448 -1.279516)
+				(xy -1.07652 -1.307792) (xy -0.98181 -1.327962) (xy -0.843334 -1.341376) (xy -0.64511 -1.349386)
+				(xy -0.371154 -1.353348) (xy -0.00548 -1.35461) (xy 0.135474 -1.354666) (xy 0.53345 -1.354028) (xy 0.834094 -1.35123)
+				(xy 1.052962 -1.344936) (xy 1.205606 -1.333816) (xy 1.307584 -1.31654) (xy 1.37445 -1.291776) (xy 1.421756 -1.258192)
+				(xy 1.43747 -1.243212) (xy 1.56739 -1.040274) (xy 1.598692 -0.806892) (xy 1.530084 -0.569812) (xy 1.474264 -0.479778)
+				(xy 1.440724 -0.442892) (xy 1.391054 -0.414356) (xy 1.31058 -0.392582) (xy 1.18463 -0.375984) (xy 0.99853 -0.36298)
+				(xy 0.737606 -0.351984) (xy 0.387182 -0.341408) (xy 0.131258 -0.334694) (xy -0.324302 -0.32141)
+				(xy -0.683016 -0.305288) (xy -0.960924 -0.2829) (xy -1.174072 -0.250812) (xy -1.338498 -0.205598)
+				(xy -1.470244 -0.143824) (xy -1.585354 -0.06206) (xy -1.699868 0.04312) (xy -1.717476 0.06062) (xy -1.903318 0.273774)
+				(xy -2.017058 0.485106) (xy -2.073562 0.732964) (xy -2.087752 1.016) (xy -2.081794 1.257778) (xy -2.055712 1.43171)
+				(xy -1.999502 1.582386) (xy -1.933434 1.703756) (xy -1.83183 1.856034) (xy 1.400446 1.856034) (xy 1.480954 1.744512)
+				(xy 1.65043 1.695054) (xy 1.69874 1.693334) (xy 1.837342 1.710132) (xy 1.904786 1.776344) (xy 1.922704 1.830372)
+				(xy 1.934886 1.988594) (xy 1.918984 2.087492) (xy 1.87127 2.167968) (xy 1.774802 2.19426) (xy 1.675028 2.190344)
+				(xy 1.523924 2.159562) (xy 1.44258 2.082602) (xy 1.416112 2.021262) (xy 1.400446 1.856034) (xy -1.83183 1.856034)
+				(xy -1.79992 1.903856) (xy -1.651946 2.060778) (xy -1.474526 2.179424) (xy -1.252674 2.264692) (xy -0.971408 2.321482)
+				(xy -0.61574 2.354696) (xy -0.170686 2.369232) (xy 0.10732 2.37104) (xy 0.476142 2.372198) (xy 0.750126 2.376504)
+				(xy 0.947318 2.385664) (xy 1.08576 2.401382) (xy 1.183492 2.425362) (xy 1.258562 2.459312) (xy 1.297794 2.483556)
+				(xy 1.500062 2.568656) (xy 1.704298 2.596074) (xy 1.868278 2.58143)
+			)
+			(stroke
+				(width 0.02)
+				(type solid)
+			)
+			(fill yes)
+			(layer "B.SilkS")
+		)
+		(embedded_fonts no)
+	)
+	(gr_text "schenktronics.com"
+		(at 157.5 100.8 0)
+		(layer "B.SilkS")
+		(effects
+			(font
+				(size 1 1)
+				(thickness 0.15)
+			)
+			(justify mirror)
+		)
+	)
+	(gr_text "ST-02 v1.0\nPassive Attenuator"
+		(at 157.5 104.0 0)
+		(layer "B.SilkS")
+		(effects
+			(font
+				(size 1 1)
+				(thickness 0.15)
+			)
+			(justify mirror)
+		)
+	)
   (gr_line (start 165 50) (end 150 50) (layer Edge.Cuts) (width 0.05))
   (gr_line (start 165 150) (end 165 50) (layer Edge.Cuts) (width 0.05))

Commit message: Main PCB: hand-tuned branding placement, add CC license text
Nathan's own edit in KiCad: refined the logo/text placement and added
"CC BY-NC-SA 4.0" text (matching the other boards -- text only, no icon
roundels). File also came back saved in modern KiCad format, which
accounts for most of this diff's size.
Parts:
- moved G*** 30.6 mm to (157.8, 67.4)
Other:
- net class Default removed
- board text added: "CC BY-NC-SA 4.0"

Commit message: Update title blocks and docs for the main PCB's silkscreen change
Nathan changed the main PCB's back silkscreen from "Passive Attenuator"
to "Levels" (ST-02 unchanged). Updates both boards' KiCad title_block
fields (still said "Passive Attenuator"/"Passive Attenuator Faceplate"),
the BOM's main-PCB label, and the assembly guide's description of what's
printed on the back.
Other:
- board text added: "ST-02 v1.0 Levels"
- board text removed: "ST-02 v1.0 Passive Attenuator"
Changed lines of the file:
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@@
 	(paper "A4")
 	(title_block
-		(title "Passive Attenuator")
+		(title "Levels")
 		(date "2026-10-07")
 		(rev "1.0")
@@
 		(0 "F.Cu" signal)
 		(2 "B.Cu" signal)
-		(9 "F.Adhes" user)
-		(11 "B.Adhes" user)
+		(9 "F.Adhes" user "F.Adhesive")
+		(11 "B.Adhes" user "B.Adhesive")
 		(13 "F.Paste" user)
 		(15 "B.Paste" user)
-		(5 "F.SilkS" user)
-		(7 "B.SilkS" user)
+		(5 "F.SilkS" user "F.Silkscreen")
+		(7 "B.SilkS" user "B.Silkscreen")
 		(1 "F.Mask" user)
 		(3 "B.Mask" user)
-		(17 "Dwgs.User" user)
-		(19 "Cmts.User" user)
-		(21 "Eco1.User" user)
-		(23 "Eco2.User" user)
+		(17 "Dwgs.User" user "User.Drawings")
+		(19 "Cmts.User" user "User.Comments")
+		(21 "Eco1.User" user "User.Eco1")
+		(23 "Eco2.User" user "User.Eco2")
 		(25 "Edge.Cuts" user)
 		(27 "Margin" user)
-		(31 "F.CrtYd" user)
-		(29 "B.CrtYd" user)
+		(31 "F.CrtYd" user "F.Courtyard")
+		(29 "B.CrtYd" user "B.Courtyard")
 		(35 "F.Fab" user)
 		(33 "B.Fab" user)
@@
 		)
 	)
-	(gr_text "ST-02 v1.0\nPassive Attenuator"
+	(gr_text "ST-02 v1.0\nLevels"
 		(at 157.5 94.8 0)
 		(layer "B.SilkS")
@@
 	)
 	(segment
+		(start 159.677001 64.677001)
+		(end 158.399999 63.399999)
+		(width 1)
+		(layer "B.Cu")
+		(net "Net-(J2-PadT)")
+	)
+	(segment
+		(start 158.399999 63.399999)
+		(end 157.5 62.5)
+		(width 1)
+		(layer "B.Cu")
+		(net "Net-(J2-PadT)")
+	)
+	(segment
+		(start 162.4 90)
+		(end 162.4 87.35)
+		(width 1)
+		(layer "B.Cu")
+		(net "Net-(J2-PadT)")
+	)
+	(segment
+		(start 162.4 87.35)
+		(end 159.677001 84.627001)
+		(width 1)
+		(layer "B.Cu")
+		(net "Net-(J2-PadT)")
+	)
+	(segment
+		(start 159.677001 84.627001)
+		(end 159.677001 64.677001)
+		(width 1)
+		(layer "B.Cu")
+		(net "Net-(J2-PadT)")
+	)
+	(segment
 		(start 163.85001 102.895992)
 		(end 163.85001 79.10001)
@@
 	)
 	(segment
-		(start 159.677001 64.677001)
-		(end 158.399999 63.399999)
+		(start 159.677001 119.677001)
+		(end 158.399999 118.399999)
 		(width 1)
 		(layer "B.Cu")
-		(net "Net-(J2-PadT)")
+		(net "Net-(J4-PadT)")
 	)
 	(segment
-		(start 158.399999 63.399999)
-		(end 157.5 62.5)
+		(start 159.677001 139.627001)
+		(end 159.677001 119.677001)
 		(width 1)
 		(layer "B.Cu")
-		(net "Net-(J2-PadT)")
+		(net "Net-(J4-PadT)")
 	)
 	(segment
-		(start 162.4 90)
-		(end 162.4 87.35)
+		(start 162.4 142.35)
+		(end 159.677001 139.627001)
 		(width 1)
 		(layer "B.Cu")
-		(net "Net-(J2-PadT)")
+		(net "Net-(J4-PadT)")
 	)
 	(segment
-		(start 162.4 87.35)
-		(end 159.677001 84.627001)
+		(start 158.399999 118.399999)
+		(end 157.5 117.5)
 		(width 1)
 		(layer "B.Cu")
-		(net "Net-(J2-PadT)")
+		(net "Net-(J4-PadT)")
 	)
 	(segment
-		(start 159.677001 84.627001)
-		(end 159.677001 64.677001)
+		(start 162.4 145)
+		(end 162.4 142.35)
 		(width 1)
 		(layer "B.Cu")
-		(net "Net-(J2-PadT)")
+		(net "Net-(J4-PadT)")
 	)
 	(segment
@@
 		(net "Net-(J3-PadT)")
 	)
-	(segment
-		(start 159.677001 119.677001)
-		(end 158.399999 118.399999)
-		(width 1)
-		(layer "B.Cu")
-		(net "Net-(J4-PadT)")
-	)
-	(segment
-		(start 159.677001 139.627001)
-		(end 159.677001 119.677001)
-		(width 1)
-		(layer "B.Cu")
-		(net "Net-(J4-PadT)")
-	)
-	(segment
-		(start 162.4 142.35)
-		(end 159.677001 139.627001)
-		(width 1)
-		(layer "B.Cu")
-		(net "Net-(J4-PadT)")
-	)
-	(segment
-		(start 158.399999 118.399999)
-		(end 157.5 117.5)
-		(width 1)
-		(layer "B.Cu")
-		(net "Net-(J4-PadT)")
-	)
-	(segment
-		(start 162.4 145)
-		(end 162.4 142.35)
-		(width 1)
-		(layer "B.Cu")
-		(net "Net-(J4-PadT)")
-	)
 	(zone
