File: PassiveAttenuatorFaceplate/PassiveAttenuatorFaceplate.kicad_pcb (KiCad board)
At the start: 2 copper layers, 15 x 128.5 mm, 9 parts

Commit message: Rename product to Levels
Faceplate silkscreen header changed from "Attenuate" to "Levels"
(ST-02 part number unchanged). Updates docs, README and the generated
panel drawings to match; renames the PDF outputs to levels-*.pdf.
The main PCB's back silkscreen still reads "Passive Attenuator", so
the assembly guide's description of it is left as-is.
Other:
- board text added: "Levels"
- board text removed: "Attenuate"
